File: schematic/keypad.kicad_sch (KiCad schematic)
At the start: 20 parts

Commit message: update schematics
Parts:
- gave numbers to parts that had none: 20
Changed lines of the file:
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@@
   (symbol (lib_id "Switch:SW_SPST") (at 130.81 78.74 0) (unit 1)
     (in_bom yes) (on_board yes) (fields_autoplaced)
-    (property "Reference" "SW?" (id 0) (at 130.81 73.3892 0))
+    (property "Reference" "SW8" (id 0) (at 130.81 73.3892 0))
     (property "Value" "2" (id 1) (at 130.81 75.9261 0))
     (property "Footprint" "" (id 2) (at 130.81 78.74 0)
@@
   (symbol (lib_id "Switch:SW_SPST") (at 184.15 109.22 0) (unit 1)
     (in_bom yes) (on_board yes) (fields_autoplaced)
-    (property "Reference" "SW?" (id 0) (at 184.15 103.8692 0))
+    (property "Reference" "SW20" (id 0) (at 184.15 103.8692 0))
     (property "Value" "C" (id 1) (at 184.15 106.4061 0))
     (property "Footprint" "" (id 2) (at 184.15 109.22 0)
@@
   (symbol (lib_id "Switch:SW_SPST") (at 130.81 93.98 0) (unit 1)
     (in_bom yes) (on_board yes) (fields_autoplaced)
-    (property "Reference" "SW?" (id 0) (at 130.81 88.6292 0))
+    (property "Reference" "SW9" (id 0) (at 130.81 88.6292 0))
     (property "Value" "5" (id 1) (at 130.81 91.1661 0))
     (property "Footprint" "" (id 2) (at 130.81 93.98 0)
@@
   (symbol (lib_id "Switch:SW_SPST") (at 104.14 93.98 0) (unit 1)
     (in_bom yes) (on_board yes) (fields_autoplaced)
-    (property "Reference" "SW?" (id 0) (at 104.14 88.6292 0))
+    (property "Reference" "SW4" (id 0) (at 104.14 88.6292 0))
     (property "Value" "4" (id 1) (at 104.14 91.1661 0))
     (property "Footprint" "" (id 2) (at 104.14 93.98 0)
@@
   (symbol (lib_id "Switch:SW_SPST") (at 157.48 63.5 0) (unit 1)
     (in_bom yes) (on_board yes) (fields_autoplaced)
-    (property "Reference" "SW?" (id 0) (at 157.48 58.1492 0))
+    (property "Reference" "SW12" (id 0) (at 157.48 58.1492 0))
     (property "Value" "P3" (id 1) (at 157.48 60.6861 0))
     (property "Footprint" "" (id 2) (at 157.48 63.5 0)
@@
   (symbol (lib_id "Switch:SW_SPST") (at 184.15 124.46 0) (unit 1)
     (in_bom yes) (on_board yes) (fields_autoplaced)
-    (property "Reference" "SW?" (id 0) (at 184.15 119.1092 0))
+    (property "Reference" "SW21" (id 0) (at 184.15 119.1092 0))
     (property "Value" "F" (id 1) (at 184.15 121.6461 0))
     (property "Footprint" "" (id 2) (at 184.15 124.46 0)
@@
   (symbol (lib_id "Switch:SW_SPST") (at 130.81 63.5 0) (unit 1)
     (in_bom yes) (on_board yes) (fields_autoplaced)
-    (property "Reference" "SW?" (id 0) (at 130.81 58.1492 0))
+    (property "Reference" "SW7" (id 0) (at 130.81 58.1492 0))
     (property "Value" "P2" (id 1) (at 130.81 60.6861 0))
     (property "Footprint" "" (id 2) (at 130.81 63.5 0)
@@
   (symbol (lib_id "Switch:SW_SPST") (at 157.48 93.98 0) (unit 1)
     (in_bom yes) (on_board yes) (fields_autoplaced)
-    (property "Reference" "SW?" (id 0) (at 157.48 88.6292 0))
+    (property "Reference" "SW14" (id 0) (at 157.48 88.6292 0))
     (property "Value" "6" (id 1) (at 157.48 91.1661 0))
     (property "Footprint" "" (id 2) (at 157.48 93.98 0)
@@
   (symbol (lib_id "Switch:SW_SPST") (at 184.15 93.98 0) (unit 1)
     (in_bom yes) (on_board yes) (fields_autoplaced)
-    (property "Reference" "SW?" (id 0) (at 184.15 88.6292 0))
+    (property "Reference" "SW19" (id 0) (at 184.15 88.6292 0))
     (property "Value" "B" (id 1) (at 184.15 91.1661 0))
     (property "Footprint" "" (id 2) (at 184.15 93.98 0)
@@
   (symbol (lib_id "Switch:SW_SPST") (at 130.81 124.46 0) (unit 1)
     (in_bom yes) (on_board yes) (fields_autoplaced)
-    (property "Reference" "SW?" (id 0) (at 130.81 119.1092 0))
+    (property "Reference" "SW11" (id 0) (at 130.81 119.1092 0))
     (property "Value" "D" (id 1) (at 130.81 121.6461 0))
     (property "Footprint" "" (id 2) (at 130.81 124.46 0)
@@
   (symbol (lib_id "Switch:SW_SPST") (at 104.14 78.74 0) (unit 1)
     (in_bom yes) (on_board yes) (fields_autoplaced)
-    (property "Reference" "SW?" (id 0) (at 104.14 73.3892 0))
+    (property "Reference" "SW3" (id 0) (at 104.14 73.3892 0))
     (property "Value" "1" (id 1) (at 104.14 75.9261 0))
     (property "Footprint" "" (id 2) (at 104.14 78.74 0)
@@
   (symbol (lib_id "Switch:SW_SPST") (at 184.15 63.5 0) (unit 1)
     (in_bom yes) (on_board yes) (fields_autoplaced)
-    (property "Reference" "SW?" (id 0) (at 184.15 58.1492 0))
+    (property "Reference" "SW17" (id 0) (at 184.15 58.1492 0))
     (property "Value" "P4" (id 1) (at 184.15 60.6861 0))
     (property "Footprint" "" (id 2) (at 184.15 63.5 0)
@@
   (symbol (lib_id "Switch:SW_SPST") (at 130.81 109.22 0) (unit 1)
     (in_bom yes) (on_board yes) (fields_autoplaced)
-    (property "Reference" "SW?" (id 0) (at 130.81 103.8692 0))
+    (property "Reference" "SW10" (id 0) (at 130.81 103.8692 0))
     (property "Value" "8" (id 1) (at 130.81 106.4061 0))
     (property "Footprint" "" (id 2) (at 130.81 109.22 0)
@@
   (symbol (lib_id "Switch:SW_SPST") (at 157.48 109.22 0) (unit 1)
     (in_bom yes) (on_board yes) (fields_autoplaced)
-    (property "Reference" "SW?" (id 0) (at 157.48 103.8692 0))
+    (property "Reference" "SW15" (id 0) (at 157.48 103.8692 0))
     (property "Value" "9" (id 1) (at 157.48 106.4061 0))
     (property "Footprint" "" (id 2) (at 157.48 109.22 0)
@@
   (symbol (lib_id "Switch:SW_SPST") (at 104.14 63.5 0) (unit 1)
     (in_bom yes) (on_board yes) (fields_autoplaced)
-    (property "Reference" "SW?" (id 0) (at 104.14 58.1492 0))
+    (property "Reference" "SW2" (id 0) (at 104.14 58.1492 0))
     (property "Value" "P1" (id 1) (at 104.14 60.6861 0))
     (property "Footprint" "" (id 2) (at 104.14 63.5 0)
@@
   (symbol (lib_id "Switch:SW_SPST") (at 104.14 124.46 0) (unit 1)
     (in_bom yes) (on_board yes) (fields_autoplaced)
-    (property "Reference" "SW?" (id 0) (at 104.14 119.1092 0))
+    (property "Reference" "SW6" (id 0) (at 104.14 119.1092 0))
     (property "Value" "0" (id 1) (at 104.14 121.6461 0))
     (property "Footprint" "" (id 2) (at 104.14 124.46 0)
@@
   (symbol (lib_id "Switch:SW_SPST") (at 184.15 78.74 0) (unit 1)
     (in_bom yes) (on_board yes) (fields_autoplaced)
-    (property "Reference" "SW?" (id 0) (at 184.15 73.3892 0))
+    (property "Reference" "SW18" (id 0) (at 184.15 73.3892 0))
     (property "Value" "A" (id 1) (at 184.15 75.9261 0))
     (property "Footprint" "" (id 2) (at 184.15 78.74 0)
@@
   (symbol (lib_id "Switch:SW_SPST") (at 157.48 124.46 0) (unit 1)
     (in_bom yes) (on_board yes) (fields_autoplaced)
-    (property "Reference" "SW?" (id 0) (at 157.48 119.1092 0))
+    (property "Reference" "SW16" (id 0) (at 157.48 119.1092 0))
     (property "Value" "E" (id 1) (at 157.48 121.6461 0))
     (property "Footprint" "" (id 2) (at 157.48 124.46 0)
@@
   (symbol (lib_id "Switch:SW_SPST") (at 157.48 78.74 0) (unit 1)
     (in_bom yes) (on_board yes) (fields_autoplaced)
-    (property "Reference" "SW?" (id 0) (at 157.48 73.3892 0))
+    (property "Reference" "SW13" (id 0) (at 157.48 73.3892 0))
     (property "Value" "3" (id 1) (at 157.48 75.9261 0))
     (property "Footprint" "" (id 2) (at 157.48 78.74 0)
@@
   (symbol (lib_id "Switch:SW_SPST") (at 104.14 109.22 0) (unit 1)
     (in_bom yes) (on_board yes) (fields_autoplaced)
-    (property "Reference" "SW?" (id 0) (at 104.14 103.8692 0))
+    (property "Reference" "SW5" (id 0) (at 104.14 103.8692 0))
     (property "Value" "7" (id 1) (at 104.14 106.4061 0))
     (property "Footprint" "" (id 2) (at 104.14 109.22 0)
