File: schematic/led_array.kicad_sch (KiCad schematic)
At the start: 16 parts

Commit message: update schematics
Parts:
- gave numbers to parts that had none: 16
Other:
- title: TEAMMATE LED Array -> T.E.A.M.M.A.T.E. LED Array
Changed lines of the file:
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@@
   (paper "A5")
   (title_block
-    (title "TEAMMATE LED Array")
+    (title "T.E.A.M.M.A.T.E. LED Array")
   )
   (junction (at 92.71 31.1439) (diameter 0) (color 0 0 0 0)
@@
   (symbol (lib_id "Device:LED") (at 142.24 72.39 0) (unit 1)
     (in_bom yes) (on_board yes) (fields_autoplaced)
-    (property "Reference" "D?" (id 0) (at 140.6525 67.4202 0)
+    (property "Reference" "D17" (id 0) (at 140.6525 67.4202 0)
       (effects (font (size 1.27 1.27)) hide)
     )
@@
   (symbol (lib_id "Device:LED") (at 124.46 52.07 0) (unit 1)
     (in_bom yes) (on_board yes) (fields_autoplaced)
-    (property "Reference" "D?" (id 0) (at 122.8725 47.1002 0)
+    (property "Reference" "D11" (id 0) (at 122.8725 47.1002 0)
       (effects (font (size 1.27 1.27)) hide)
     )
@@
   (symbol (lib_id "Device:LED") (at 106.68 52.07 0) (unit 1)
     (in_bom yes) (on_board yes) (fields_autoplaced)
-    (property "Reference" "D?" (id 0) (at 105.0925 47.1002 0)
+    (property "Reference" "D7" (id 0) (at 105.0925 47.1002 0)
       (effects (font (size 1.27 1.27)) hide)
     )
@@
   (symbol (lib_id "Device:LED") (at 106.68 41.91 0) (unit 1)
     (in_bom yes) (on_board yes) (fields_autoplaced)
-    (property "Reference" "D?" (id 0) (at 105.0925 36.9402 0)
+    (property "Reference" "D6" (id 0) (at 105.0925 36.9402 0)
       (effects (font (size 1.27 1.27)) hide)
     )
@@
   (symbol (lib_id "Device:LED") (at 142.24 52.07 0) (unit 1)
     (in_bom yes) (on_board yes) (fields_autoplaced)
-    (property "Reference" "D?" (id 0) (at 140.6525 47.1002 0)
+    (property "Reference" "D15" (id 0) (at 140.6525 47.1002 0)
       (effects (font (size 1.27 1.27)) hide)
     )
@@
   (symbol (lib_id "Device:LED") (at 124.46 72.39 0) (unit 1)
     (in_bom yes) (on_board yes) (fields_autoplaced)
-    (property "Reference" "D?" (id 0) (at 122.8725 67.4202 0)
+    (property "Reference" "D13" (id 0) (at 122.8725 67.4202 0)
       (effects (font (size 1.27 1.27)) hide)
     )
@@
   (symbol (lib_id "Device:LED") (at 124.46 62.23 0) (unit 1)
     (in_bom yes) (on_board yes) (fields_autoplaced)
-    (property "Reference" "D?" (id 0) (at 122.8725 57.2602 0)
+    (property "Reference" "D12" (id 0) (at 122.8725 57.2602 0)
       (effects (font (size 1.27 1.27)) hide)
     )
@@
   (symbol (lib_id "Device:LED") (at 124.46 41.91 0) (unit 1)
     (in_bom yes) (on_board yes) (fields_autoplaced)
-    (property "Reference" "D?" (id 0) (at 122.8725 36.9402 0)
+    (property "Reference" "D10" (id 0) (at 122.8725 36.9402 0)
       (effects (font (size 1.27 1.27)) hide)
     )
@@
   (symbol (lib_id "Device:LED") (at 88.9 52.07 0) (unit 1)
     (in_bom yes) (on_board yes) (fields_autoplaced)
-    (property "Reference" "D?" (id 0) (at 87.3125 47.1002 0)
+    (property "Reference" "D3" (id 0) (at 87.3125 47.1002 0)
       (effects (font (size 1.27 1.27)) hide)
     )
@@
   (symbol (lib_id "Device:LED") (at 88.9 72.39 0) (unit 1)
     (in_bom yes) (on_board yes) (fields_autoplaced)
-    (property "Reference" "D?" (id 0) (at 87.3125 67.4202 0)
+    (property "Reference" "D5" (id 0) (at 87.3125 67.4202 0)
       (effects (font (size 1.27 1.27)) hide)
     )
@@
   (symbol (lib_id "Device:LED") (at 88.9 62.23 0) (unit 1)
     (in_bom yes) (on_board yes) (fields_autoplaced)
-    (property "Reference" "D?" (id 0) (at 87.3125 57.2602 0)
+    (property "Reference" "D4" (id 0) (at 87.3125 57.2602 0)
       (effects (font (size 1.27 1.27)) hide)
     )
@@
   (symbol (lib_id "Device:LED") (at 88.9 41.91 0) (unit 1)
     (in_bom yes) (on_board yes) (fields_autoplaced)
-    (property "Reference" "D?" (id 0) (at 87.3125 36.9402 0)
+    (property "Reference" "D2" (id 0) (at 87.3125 36.9402 0)
       (effects (font (size 1.27 1.27)) hide)
     )
@@
   (symbol (lib_id "Device:LED") (at 106.68 62.23 0) (unit 1)
     (in_bom yes) (on_board yes) (fields_autoplaced)
-    (property "Reference" "D?" (id 0) (at 105.0925 57.2602 0)
+    (property "Reference" "D8" (id 0) (at 105.0925 57.2602 0)
       (effects (font (size 1.27 1.27)) hide)
     )
@@
   (symbol (lib_id "Device:LED") (at 142.24 62.23 0) (unit 1)
     (in_bom yes) (on_board yes) (fields_autoplaced)
-    (property "Reference" "D?" (id 0) (at 140.6525 57.2602 0)
+    (property "Reference" "D16" (id 0) (at 140.6525 57.2602 0)
       (effects (font (size 1.27 1.27)) hide)
     )
@@
   (symbol (lib_id "Device:LED") (at 106.68 72.39 0) (unit 1)
     (in_bom yes) (on_board yes) (fields_autoplaced)
-    (property "Reference" "D?" (id 0) (at 105.0925 67.4202 0)
+    (property "Reference" "D9" (id 0) (at 105.0925 67.4202 0)
       (effects (font (size 1.27 1.27)) hide)
     )
@@
   (symbol (lib_id "Device:LED") (at 142.24 41.91 0) (unit 1)
     (in_bom yes) (on_board yes) (fields_autoplaced)
-    (property "Reference" "D?" (id 0) (at 140.6525 36.9402 0)
-      (effects (font (size 1.27 1.27)) hide)
-    )
+    (property "Reference" "D14" (id 0) (at 140.6525 36.9402 0)
+      (effects (font (size 1.27 1.27)) hide)
+    )
